File: keyboard-pcb-tutorial.sch (KiCad schematic (older format))
At the start: 14 parts

Commit message: Finish schematic, add footprints
Parts:
- added D1, D2, D3, D4: D_Small, Diode_SMD:D_SOD-123, symbol Device:D_Small
- added F1, F2: 500mA, Fuse:Fuse_1206_3216Metric, symbol Device:Polyfuse_Small
- added MX1, MX2, MX3, MX4: MX-NoLED, MX_Alps_Hybrid:MX-1U-NoLED, symbol MX_Alps_Hybrid:MX-NoLED
- added USB1: Molex-0548190589, random-keyboard-parts:Molex-0548190589, symbol random-keyboard-parts:Molex-0548190589
- C1, C2, C3, C4, C5, C6, C7: renamed from C?; footprint (none) -> Capacitor_SMD:C_0805_2012Metric
- R1, R2, R3, R4: renamed from R?; footprint (none) -> Resistor_SMD:R_0805_2012Metric
- SW1: renamed from SW?; footprint (none) -> random-keyboard-parts:SKQG-1155865
- Y1: renamed from Y?; footprint (none) -> Crystal:Crystal_SMD_3225-4Pin_3.2x2.5mm
- gave numbers to parts that had none: 1
Connections:
- net +5V: now also F1.2, F2.1; no longer U1.7 (VBUS)
- net D+: now also USB1.3 (D+)
- net D-: now also USB1.4 (D-)
- net GND: now also USB1.1 (GND)
- new net: D3.2 (A), MX3.2 (ROW)
- new net: D4.2 (A), MX4.2 (ROW)
- new net: D1.2 (A), MX1.2 (ROW)
- new net: D2.2 (A), MX2.2 (ROW)
- new net COL0: MX1.1 (COL), MX3.1 (COL)
- new net COL1: MX2.1 (COL), MX4.1 (COL)
- new net ROW0: D1.1 (K), D2.1 (K)
- new net ROW1: D3.1 (K), D4.1 (K)
- new net VCC: F1.1, F2.2, U1.7 (VBUS), USB1.5 (VBUS)

Commit message: route pcb
Connections:
- net COL0: now also U1.29 (PB5)
- net COL1: now also U1.28 (PB4)
- net ROW0: now also U1.27 (PD7)
- net ROW1: now also U1.30 (PB6)
Changed lines of the file:
@@
 	0    1    1    0
 $EndComp
-$Comp
-L power:VCC #PWR0111
-U 1 1 628E2AB7
-P 4400 3500
-F 0 "#PWR0111" H 4400 3350 50  0001 C CNN
-F 1 "VCC" H 4417 3673 50  0000 C CNN
-F 2 "" H 4400 3500 50  0001 C CNN
-F 3 "" H 4400 3500 50  0001 C CNN
-	1    4400 3500
-	1    0    0    -1
-$EndComp
 Wire Wire Line
 	4400 3500 4350 3500
-Connection ~ 4400 3500
 Wire Wire Line
 	4150 3500 4100 3500
@@
 Text GLabel 6750 3100 0    50   Input ~ 0
 ROW1
+Connection ~ 4400 3500
+$Comp
+L power:VCC #PWR0111
+U 1 1 628E2AB7
+P 4400 3500
+F 0 "#PWR0111" H 4400 3350 50  0001 C CNN
+F 1 "VCC" H 4417 3673 50  0000 C CNN
+F 2 "" H 4400 3500 50  0001 C CNN
+F 3 "" H 4400 3500 50  0001 C CNN
+	1    4400 3500
+	1    0    0    -1
+$EndComp
+Text GLabel 5600 3300 2    50   Input ~ 0
+ROW1
+Text GLabel 5600 3200 2    50   Input ~ 0
+COL0
+Text GLabel 5600 3100 2    50   Input ~ 0
+COL1
+Text GLabel 5600 4600 2    50   Input ~ 0
+ROW0
 $EndSCHEMATC
