File: keyboard-pcb-tutorial.kicad_pcb (KiCad board)
At the start: 2 copper layers, 77 x 38.1 mm, 25 parts, among them SW1 SW_Push, U1 ATmega32U4-AU, Y1 16MHz

Commit message: route pcb
Parts:
- moved C7 6.78 mm to (107.2, 108.0), turned to 90 degrees
- moved F1 1.59 mm to (108.0, 99.2)
- moved R2 1.59 mm to (99.2, 95.2)
- moved C3 0.97 mm to (108.0, 102.4), turned to 0 degrees
Connections:
- U1 pad 27: Net-(U1-Pad27) -> ROW0
- U1 pad 28: Net-(U1-Pad28) -> COL1
- U1 pad 29: Net-(U1-Pad29) -> COL0
- U1 pad 30: Net-(U1-Pad30) -> ROW1
Routing:
- net GND: track 0.00 -> 138.0 mm
- net +5V: track 0.00 -> 113.7 mm, vias 0 -> 5
- net COL1: track 0.00 -> 53.3 mm
- net ROW1: track 0.00 -> 50.7 mm
- net ROW0: track 0.00 -> 46.9 mm
- net VCC: track 0.00 -> 34.7 mm
- net Net-(R1-Pad2): track 0.00 -> 34.5 mm, vias 0 -> 2
- net COL0: track 0.00 -> 33.9 mm
- net Net-(R3-Pad1): track 0.00 -> 19.4 mm
- net Net-(R2-Pad1): track 0.00 -> 15.9 mm
- net Net-(C2-Pad1): track 0.00 -> 13.4 mm
- net Net-(C1-Pad1): track 0.00 -> 10.6 mm
- net Net-(D2-Pad2): track 0.00 -> 6.82 mm
- net Net-(D3-Pad2): track 0.00 -> 6.82 mm
- net Net-(D1-Pad2): track 0.00 -> 6.82 mm
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Other:
- net class Default: trace_width 0.25 -> 0.254
- net class Power added: clearance 0.2, trace_width 0.381, via_dia 0.8, via_drill 0.4

Commit message: Finish PCB
Parts:
- moved C3 1.12 mm to (108.7, 101.6), turned to 180 degrees
- moved C4 0.95 mm to (110.3, 92.9)
Routing:
- net Net-(USB1-Pad6): track 0.00 -> 16.3 mm
- net GND: track 138.0 -> 142.1 mm, vias 0 -> 2
- net +5V: track 113.7 -> 109.7 mm
- net Net-(C3-Pad1): track 5.70 -> 2.64 mm
- net Net-(R2-Pad1): track 15.9 -> 16.9 mm
- added copper zone on B.Cu, net GND
Other:
- board size 77 x 38.1 mm -> 77.8 x 38.1 mm
